Commit message: Mitsubishi arm controller is now working

File: mitsubishi_arm_description/robots/mitsubishi_rv_6sdl_barret.urdf.xacro (robot description, xacro)
@@ -2,11 +2,11 @@
 <robot xmlns:xacro="http://ros.org/wiki/xacro" name="mitsubishi_and_barret">
   <!-- LINKS   -->
-  <xacro:include filename="$(find mitsubishi_rv_6sdl_description)/urdf/mitsubishi_rv_6sdl_arm.urdf.xacro" />
-  <joint name="arm_to_gripper" type="fixed">
+  <xacro:include filename="$(find mitsubishi_arm_description)/urdf/mitsubishi_rv_6sdl_arm.urdf.xacro" />
+  <!--<joint name="arm_to_gripper" type="fixed">
     <parent link="end_effector" />
     <child link="barret_base_link" />
     <axis xyz="0 0 1" />
     <limit lower="-3.141" upper="0" effort="0" velocity="0" />
-  </joint>
-  <xacro:include filename="$(find barret_hand_description)/robots/bhand_model.URDF" />
+  </joint>-->
+  <!--<xacro:include filename="$(find barret_hand_description)/robots/bhand_model.URDF" />-->
 </robot>

Commit message: mitsubishi arm hardware interface new tests...

File: mitsubishi_arm_description/robots/mitsubishi_rv_6sdl_barret.urdf.xacro (robot description, xacro)
@@ -5,8 +5,8 @@
   <joint name="arm_to_gripper" type="fixed">
     <parent link="end_effector" />
-    <child link="barret_base_link" />
+    <child link="barrett_base_link" />
     <axis xyz="0 0 1" />
     <limit lower="-3.141" upper="0" effort="0" velocity="0" />
   </joint>
-  <xacro:include filename="$(find barret_hand_description)/robots/bhand_model.URDF" />
+  <xacro:include filename="$(find barrett_hand_description)/robots/bhand_model.URDF" />
 </robot>
