Commit message: mitsubishi arm working in gazebo with kinect sensor

File: mitsubishi_arm_description/robots/mitsubishi_rv_6sdl_gazebo.urdf.xacro (robot description, xacro)
@@ -33,5 +33,5 @@
   <!--<xacro:include filename="$(find mitsubishi_arm_description)/urdf/sensors.xacro" />-->
   <!-- kinect to base link -->
- <!-- <joint name="camera_in_world_joint" type="fixed">
+  <!--<joint name="camera_in_world_joint" type="fixed">
     <parent link="base_link"/>
     <child link="camera_link"/>
