Commit message: mitsubishi arm now works in gazebo

File: mitsubishi_arm_description/robots/mitsubishi_rv_6sdl.urdf.xacro (robot description, xacro)
@@ -1,4 +1,14 @@
 <?xml version="1.0"?>
 <robot xmlns:xacro="http://ros.org/wiki/xacro" name="mitsubishi_arm">
+  <!-- Import all Gazebo-customization elements, including Gazebo colors -->
+  <xacro:include filename="$(find mitsubishi_arm_description)/urdf/mitsubishi_rv_6sdl_arm.gazebo" />
+  <!-- Import Rviz colors -->
+  <xacro:include filename="$(find rrbot_description)/urdf/materials.xacro" />
+  <!-- Used for fixing robot to Gazebo 'base_link' -->
+  <link name="world"/>
+  <joint name="fixed" type="fixed">
+    <parent link="world"/>
+    <child link="base_link"/>
+  </joint>
   <!-- LINKS   -->
   <xacro:include filename="$(find mitsubishi_arm_description)/urdf/mitsubishi_rv_6sdl_arm.xacro" />

File: mitsubishi_arm_description/urdf/mitsubishi_rv_6sdl_arm.xacro (robot description, xacro)
@@ -3,4 +3,5 @@
   <property name="PI" value="3.1415926535897931" />
   <property name="offset_from_limit" value="5.0" />
+  <!-- base_link -->
   <link name="base_link" >
     <visual>
@@ -19,4 +20,12 @@
       <origin xyz="-0.1125 0 .1185"/>
     </collision>
+    <inertial>
+      <origin xyz="0 0 1" rpy="0 0 0"/>
+      <mass value="0.01"/>
+      <inertia
+        ixx="1.0" ixy="0.0" ixz="0.0"
+        iyy="1.0" iyz="0.0"
+        izz="1.0"/>
+    </inertial>
   </link>
   <joint name="j1" type="revolute">
@@ -26,5 +35,7 @@
     <child link="shoulder_block"/>
     <origin xyz="0 0 0.239"/>
-  </joint>
+    <dynamics damping="0.0"/>
+  </joint>
+  <!-- shoulder_block -->
   <link name="shoulder_block">
     <visual>
@@ -43,4 +54,12 @@
       <origin xyz="-.100 0 0.0555"/>
     </collision>
+    <inertial>
+      <origin xyz="0 0 1" rpy="0 0 0"/>
+      <mass value="0.01"/>
+      <inertia
+        ixx="1.0" ixy="0.0" ixz="0.0"
+        iyy="1.0" iyz="0.0"
+        izz="1.0"/>
+    </inertial>
   </link>
   <joint name="j2" type="revolute">
@@ -50,5 +69,7 @@
     <child link="shoulder"/>
     <origin xyz="0.079 0 0.111" rpy="1.57079632679 0 3.14159265359"/>
-  </joint>
+    <dynamics damping="0.0"/>
+  </joint>
+  <!-- shoulder -->
   <link name="shoulder">
     <visual>
@@ -67,4 +88,12 @@
       <origin xyz="0 0 0"/>
     </collision>
+    <inertial>
+      <origin xyz="0 0 1" rpy="0 0 0"/>
+      <mass value="0.01"/>
+      <inertia
+        ixx="1.0" ixy="0.0" ixz="0.0"
+        iyy="1.0" iyz="0.0"
+        izz="1.0"/>
+    </inertial>
   </link>
   <joint name="fixed_joint_1" type="fixed">
@@ -73,5 +102,7 @@
     <child link="upper_arm"/>
     <origin xyz="0 0.079 0"/>
-  </joint>
+    <dynamics damping="0.0"/>
+  </joint>
+  <!-- upper_arm -->
   <link name="upper_arm">
     <visual>
@@ -90,4 +121,12 @@
       <origin xyz="0 0.111 0.102"/>
     </collision>
+    <inertial>
+      <origin xyz="0 0 1" rpy="0 0 0"/>
+      <mass value="0.01"/>
+      <inertia
+        ixx="1.0" ixy="0.0" ixz="0.0"
+        iyy="1.0" iyz="0.0"
+        izz="1.0"/>
+    </inertial>
   </link>
   <joint name="j3" type="revolute">
@@ -97,5 +136,7 @@
     <child link="elbow"/>
     <origin xyz="0 0.301 0" rpy="0 0 1.57"/>
-  </joint>
+    <dynamics damping="0.0"/>
+  </joint>
+  <!-- elbow -->
   <link name="elbow">
     <visual>
@@ -114,4 +155,12 @@
       <origin xyz="0 0 0"/>
     </collision>
+    <inertial>
+      <origin xyz="0 0 1" rpy="0 0 0"/>
+      <mass value="0.01"/>
+      <inertia
+        ixx="1.0" ixy="0.0" ixz="0.0"
+        iyy="1.0" iyz="0.0"
+        izz="1.0"/>
+    </inertial>
   </link>
   <joint name="fixed_joint_2" type="fixed">
@@ -119,5 +168,7 @@
     <child link="elbow_block"/>
     <origin xyz="0 -0.100 0"/>
-  </joint>
+    <dynamics damping="0.0"/>
+  </joint>
+  <!-- elbow_block -->
   <link name="elbow_block">
     <visual>
@@ -136,4 +187,12 @@
       <origin xyz="-0.0275 0 0"/>
     </collision>
+    <inertial>
+      <origin xyz="0 0 1" rpy="0 0 0"/>
+      <mass value="0.01"/>
+      <inertia
+        ixx="1.0" ixy="0.0" ixz="0.0"
+        iyy="1.0" iyz="0.0"
+        izz="1.0"/>
+    </inertial>
   </link>
   <joint name="j4" type="revolute">
@@ -143,5 +202,7 @@
     <child link="fore_arm"/>
     <origin xyz="0.079 0 0"  rpy="0 1.5707963267 0"/>
-  </joint>
+    <dynamics damping="0.0"/>
+  </joint>
+  <!-- fore_arm -->
   <link name="fore_arm">
     <visual>
@@ -160,4 +221,12 @@
       <origin xyz="0 0 0.1815"/>
     </collision>
+    <inertial>
+      <origin xyz="0 0 1" rpy="0 0 0"/>
+      <mass value="0.01"/>
+      <inertia
+        ixx="1.0" ixy="0.0" ixz="0.0"
+        iyy="1.0" iyz="0.0"
+        izz="1.0"/>
+    </inertial>
   </link>
   <joint name="j5" type="revolute">
@@ -167,5 +236,7 @@
     <child link="wrist"/>
     <origin xyz="0 0 0.346"  rpy="0.0 -1.5707963267 0"/>
-  </joint>
+    <dynamics damping="0.0"/>
+  </joint>
+  <!-- wrist -->
   <link name="wrist">
     <visual>
@@ -184,4 +255,12 @@
       <origin xyz="0 0 0"/>
     </collision>
+    <inertial>
+      <origin xyz="0 0 1" rpy="0 0 0"/>
+      <mass value="0.01"/>
+      <inertia
+        ixx="1.0" ixy="0.0" ixz="0.0"
+        iyy="1.0" iyz="0.0"
+        izz="1.0"/>
+    </inertial>
   </link>
   <joint name="j6" type="revolute">
@@ -191,5 +270,7 @@
     <child link="torque_sensor"/>
     <origin xyz="0.085 0 0"  rpy="0 1.5707963267 0"/>
-  </joint>
+    <dynamics damping="0.0"/>
+  </joint>
+  <!-- torque_sensor -->
   <link name="torque_sensor">
     <visual>
@@ -211,4 +292,12 @@
       </material>
     </collision>
+    <inertial>
+      <origin xyz="0 0 1" rpy="0 0 0"/>
+      <mass value="0.01"/>
+      <inertia
+        ixx="1.0" ixy="0.0" ixz="0.0"
+        iyy="1.0" iyz="0.0"
+        izz="1.0"/>
+    </inertial>
   </link>
   <joint name="torque_sensor_joint" type="fixed">
@@ -218,6 +307,64 @@
     <child link="end_effector"/>
     <origin xyz="0 0 0.065"  rpy="0 0 0"/> <!-- original is 0.085 but we have the torque sensor...-->
-  </joint>
+    <dynamics damping="0.0"/>
+  </joint>
+  <!-- end_effector -->
   <link name="end_effector">
-  </link>
+    <inertial>
+      <origin xyz="0 0 1" rpy="0 0 0"/>
+      <mass value="0.01"/>
+      <inertia
+        ixx="1.0" ixy="0.0" ixz="0.0"
+        iyy="1.0" iyz="0.0"
+        izz="1.0"/>
+    </inertial>
+  </link>
+  <transmission name="tran1">
+    <type>transmission_interface/SimpleTransmission</type>
+    <joint name="j1"/>
+    <actuator name="motor1">
+      <hardwareInterface>EffortJointInterface</hardwareInterface>
+      <mechanicalReduction>1</mechanicalReduction>
+    </actuator>
+  </transmission>
+  <transmission name="tran2">
+    <type>transmission_interface/SimpleTransmission</type>
+    <joint name="j2"/>
+    <actuator name="motor2">
+      <hardwareInterface>EffortJointInterface</hardwareInterface>
+      <mechanicalReduction>1</mechanicalReduction>
+    </actuator>
+  </transmission>
+  <transmission name="tran3">
+    <type>transmission_interface/SimpleTransmission</type>
+    <joint name="j3"/>
+    <actuator name="motor3">
+      <hardwareInterface>EffortJointInterface</hardwareInterface>
+      <mechanicalReduction>1</mechanicalReduction>
+    </actuator>
+  </transmission>
+  <transmission name="tran4">
+    <type>transmission_interface/SimpleTransmission</type>
+    <joint name="j4"/>
+    <actuator name="motor4">
+      <hardwareInterface>EffortJointInterface</hardwareInterface>
+      <mechanicalReduction>1</mechanicalReduction>
+    </actuator>
+  </transmission>
+  <transmission name="tran5">
+    <type>transmission_interface/SimpleTransmission</type>
+    <joint name="j5"/>
+    <actuator name="motor5">
+      <hardwareInterface>EffortJointInterface</hardwareInterface>
+      <mechanicalReduction>1</mechanicalReduction>
+    </actuator>
+  </transmission>
+  <transmission name="tran6">
+    <type>transmission_interface/SimpleTransmission</type>
+    <joint name="j6"/>
+    <actuator name="motor6">
+      <hardwareInterface>EffortJointInterface</hardwareInterface>
+      <mechanicalReduction>1</mechanicalReduction>
+    </actuator>
+  </transmission>
 </robot>

Commit message: added files regarding barrett hand in gazebo (still not working though)

File: mitsubishi_arm_description/robots/mitsubishi_rv_6sdl.urdf.xacro (robot description, xacro)
@@ -4,5 +4,19 @@
   <xacro:include filename="$(find mitsubishi_arm_description)/urdf/mitsubishi_rv_6sdl_arm.gazebo" />
   <!-- Import Rviz colors -->
-  <xacro:include filename="$(find rrbot_description)/urdf/materials.xacro" />
+  <xacro:include filename="$(find mitsubishi_arm_description)/urdf/materials.xacro" />
+  <!-- ros_control plugin -->
+  <gazebo>
+    <plugin name="gazebo_ros_control" filename="libgazebo_ros_control.so">
+      <robotNamespace>/mitsubishi_arm</robotNamespace>
+      <robotSimType>gazebo_ros_control/DefaultRobotHWSim</robotSimType>
+    </plugin>
+  </gazebo>
+  <gazebo>
+    <plugin name="gazebo_ros_joint_trajectory" filename="libgazebo_ros_joint_pose_trajectory.so">
+      <robotNamespace>/mitsubishi_arm</robotNamespace>
+      <alwaysOn>true</alwaysOn>
+      <updateRate>100.0</updateRate>
+    </plugin>
+  </gazebo>
   <!-- Used for fixing robot to Gazebo 'base_link' -->
   <link name="world"/>

File: mitsubishi_arm_description/urdf/mitsubishi_rv_6sdl_arm.xacro (robot description, xacro)
@@ -35,5 +35,5 @@
     <child link="shoulder_block"/>
     <origin xyz="0 0 0.239"/>
-    <dynamics damping="0.0"/>
+   <dynamics damping="100.0" friction="100.0" />
   </joint>
   <!-- shoulder_block -->
@@ -69,5 +69,5 @@
     <child link="shoulder"/>
     <origin xyz="0.079 0 0.111" rpy="1.57079632679 0 3.14159265359"/>
-    <dynamics damping="0.0"/>
+   <dynamics damping="100.0" friction="100.0" />
   </joint>
   <!-- shoulder -->
@@ -102,5 +102,5 @@
     <child link="upper_arm"/>
     <origin xyz="0 0.079 0"/>
-    <dynamics damping="0.0"/>
+   <dynamics damping="100.0" friction="100.0" />
   </joint>
   <!-- upper_arm -->
@@ -136,5 +136,5 @@
     <child link="elbow"/>
     <origin xyz="0 0.301 0" rpy="0 0 1.57"/>
-    <dynamics damping="0.0"/>
+   <dynamics damping="100.0" friction="100.0" />
   </joint>
   <!-- elbow -->
@@ -168,5 +168,5 @@
     <child link="elbow_block"/>
     <origin xyz="0 -0.100 0"/>
-    <dynamics damping="0.0"/>
+   <dynamics damping="100.0" friction="100.0" />
   </joint>
   <!-- elbow_block -->
@@ -202,5 +202,5 @@
     <child link="fore_arm"/>
     <origin xyz="0.079 0 0"  rpy="0 1.5707963267 0"/>
-    <dynamics damping="0.0"/>
+   <dynamics damping="100.0" friction="100.0" />
   </joint>
   <!-- fore_arm -->
@@ -236,5 +236,5 @@
     <child link="wrist"/>
     <origin xyz="0 0 0.346"  rpy="0.0 -1.5707963267 0"/>
-    <dynamics damping="0.0"/>
+   <dynamics damping="100.0" friction="100.0" />
   </joint>
   <!-- wrist -->
@@ -270,5 +270,5 @@
     <child link="torque_sensor"/>
     <origin xyz="0.085 0 0"  rpy="0 1.5707963267 0"/>
-    <dynamics damping="0.0"/>
+   <dynamics damping="10.0" friction="100.0" />
   </joint>
   <!-- torque_sensor -->
@@ -307,5 +307,5 @@
     <child link="end_effector"/>
     <origin xyz="0 0 0.065"  rpy="0 0 0"/> <!-- original is 0.085 but we have the torque sensor...-->
-    <dynamics damping="0.0"/>
+   <dynamics damping="100.0" friction="100.0" />
   </joint>
   <!-- end_effector -->

Commit message: started calibrating kinect transformation to the mitsubishi arm base link. de

File: mitsubishi_arm_description/robots/mitsubishi_rv_6sdl.urdf.xacro (robot description, xacro)
@@ -1,4 +1,7 @@
 <?xml version="1.0"?>
 <robot xmlns:xacro="http://ros.org/wiki/xacro" name="mitsubishi_arm">
+  <property name="table_y_length" value="1.0" />
+  <property name="camera_table_y_offset" value="0.265" />
+  <property name="camera_table_x_offset" value="1.0" />
   <!-- Import all Gazebo-customization elements, including Gazebo colors -->
   <xacro:include filename="$(find mitsubishi_arm_description)/urdf/mitsubishi_rv_6sdl_arm.gazebo" />
@@ -27,3 +30,12 @@
   <!-- LINKS   -->
   <xacro:include filename="$(find mitsubishi_arm_description)/urdf/mitsubishi_rv_6sdl_arm.xacro" />
+  <!-- Kinect -->
+  <xacro:include filename="$(find mitsubishi_arm_description)/urdf/sensors.xacro" />
+  <link name="arm_to_kinect">
+  </link>
+  <joint name="arm_camera" type="fixed">
+    <parent link="base_link"/>
+    <child link="arm_to_kinect"/>
+    <origin xyz="0.50 ${table_y_length/2.0 + camera_table_y_offset} 0" rpy="0 0 0"/>
+  </joint>
 </robot>

Commit message: mitsubishi is being calibrated with ar markers but still needs some tuning. Needs to use a batch of markers

File: mitsubishi_arm_description/robots/mitsubishi_rv_6sdl.urdf.xacro (robot description, xacro)
@@ -32,10 +32,16 @@
   <!-- Kinect -->
   <xacro:include filename="$(find mitsubishi_arm_description)/urdf/sensors.xacro" />
-  <link name="arm_to_kinect">
+  <!--<link name="camera_rgb_optical_frame">
   </link>
-  <joint name="arm_camera" type="fixed">
-    <parent link="base_link"/>
-    <child link="arm_to_kinect"/>
-    <origin xyz="0.50 ${table_y_length/2.0 + camera_table_y_offset} 0" rpy="0 0 0"/>
+  <joint name="camera_in_world_joint" type="fixed">
+    <parent link="world"/>
+    <child link="camera_rgb_optical_frame"/>
   </joint>
+  <link name="camera_to_marker">
+  </link>
+  <joint name="camera_to_marker_joint" type="fixed">
+    <parent link="camera_rgb_optical_frame"/>
+    <child link="camera_to_marker"/>
+    <origin xyz="0.653 0.135 -0.17" rpy="-3.04074 -1.19202 -1.6786"/>
+  </joint>-->
 </robot>

File: mitsubishi_arm_description/urdf/mitsubishi_rv_6sdl_arm.xacro (robot description, xacro)
@@ -276,5 +276,5 @@
     <visual>
      <geometry>
-	<cylinder  length="0.065" radius="0.035"/>
+	<cylinder  length="0.065" radius="0.065"/>
       </geometry>
       <origin xyz="0 0 0.0325"/>
@@ -285,5 +285,5 @@
     <collision>
      <geometry>
-	<cylinder  length="0.065" radius="0.035"/>
+	<cylinder  length="0.065" radius="0.065"/>
       </geometry>
       <origin xyz="0 0 0.0325"/>

Commit message: debugging barrett hand velocity controller with effort feedback

File: mitsubishi_arm_description/robots/mitsubishi_rv_6sdl.urdf.xacro (robot description, xacro)
@@ -32,16 +32,9 @@
   <!-- Kinect -->
   <xacro:include filename="$(find mitsubishi_arm_description)/urdf/sensors.xacro" />
-  <!--<link name="camera_rgb_optical_frame">
-  </link>
+  <!-- kinect to base link -->
   <joint name="camera_in_world_joint" type="fixed">
-    <parent link="world"/>
-    <child link="camera_rgb_optical_frame"/>
+    <parent link="base_link"/>
+    <child link="camera_link"/>
+    <origin xyz="0.796357 0.919602 0.431341" rpy="0.0247013 0.415733 -1.55723"/>
   </joint>
-  <link name="camera_to_marker">
-  </link>
-  <joint name="camera_to_marker_joint" type="fixed">
-    <parent link="camera_rgb_optical_frame"/>
-    <child link="camera_to_marker"/>
-    <origin xyz="0.653 0.135 -0.17" rpy="-3.04074 -1.19202 -1.6786"/>
-  </joint>-->
 </robot>

File: mitsubishi_arm_description/urdf/sensors.xacro (robot description, xacro)
@@ -3,4 +3,5 @@
   <property name="PI" value="3.1415926535897931" />
   <property name="offset_from_limit" value="5.0" />
-  <!-- shoulder_block -->
+  <link name="camera_link">
+  </link>
 </robot>

Commit message: latest version for the demo

File: mitsubishi_arm_description/robots/mitsubishi_rv_6sdl.urdf.xacro (robot description, xacro)
@@ -30,4 +30,56 @@
   <!-- LINKS   -->
   <xacro:include filename="$(find mitsubishi_arm_description)/urdf/mitsubishi_rv_6sdl_arm.xacro" />
+`
+  <joint name="end_effector_to_gripper_palm" type="fixed">
+    <axis xyz="0 0 1"/>
+    <limit effort="1000.0" lower="${(-360+offset_from_limit)*PI/180}" upper="${(360-offset_from_limit)*PI/180}" velocity="0.2"/>
+    <parent link="end_effector"/>
+    <child link="palm_frame"/>
+    <origin xyz="0 0 0.065"  rpy="0 0 0"/> <!-- original is 0.085 but we have the torque sensor...-->
+   <dynamics damping="100.0" friction="100.0" />
+  </joint>
+  <!-- end_effector -->
+  <link name="palm_frame">
+    <inertial>
+      <origin xyz="0 0 1" rpy="0 0 0"/>
+      <mass value="0.01"/>
+      <inertia
+        ixx="1.0" ixy="0.0" ixz="0.0"
+        iyy="1.0" iyz="0.0"
+        izz="1.0"/>
+    </inertial>
+  </link>
+  <joint name="finger_1_joint" type="fixed">
+    <axis xyz="0 0 1"/>
+    <parent link="palm_frame"/>
+    <child link="finger_1"/>
+    <origin xyz="0 0 0"  rpy="0 0 1.56"/> <!-- original is 0.085 but we have the torque sensor...-->
+   <dynamics damping="100.0" friction="100.0" />
+  </joint>
+  <link name="finger_1">
+    <visual>
+     <geometry>
+	<box size="0.350 .05 .02"/>
+      </geometry>
+      <origin xyz="0 0 -0.011"/>
+      <material name="orange">
+        <color rgba="1 1 1 1"/>
+      </material>
+    </visual>
+    <collision>
+     <geometry>
+	<box size="0.350 .05 .02"/>
+      </geometry>
+      <origin xyz="0 0 -0.011"/>
+    </collision>
+    <inertial>
+      <origin xyz="0 0 1" rpy="0 0 0"/>
+      <mass value="0.01"/>
+      <inertia
+        ixx="1.0" ixy="0.0" ixz="0.0"
+        iyy="1.0" iyz="0.0"
+        izz="1.0"/>
+    </inertial>
+  </link>
   <!-- Kinect -->
   <!--<xacro:include filename="$(find mitsubishi_arm_description)/urdf/sensors.xacro" />-->

File: mitsubishi_arm_description/urdf/mitsubishi_rv_6sdl_arm.xacro (robot description, xacro)
@@ -10,5 +10,5 @@
       </geometry>
       <origin xyz="-0.1125 0 .1185"/>
-      <material name="white">
+      <material name="orange">
         <color rgba="1 1 1 1"/>
       </material>
@@ -44,5 +44,5 @@
       </geometry>
       <origin xyz="-.100 0 0.0555"/>
-      <material name="white">
+      <material name="orange">
         <color rgba="1 1 1 1"/>
       </material>
@@ -78,5 +78,5 @@
       </geometry>
       <origin xyz="0 0 0"/>
-      <material name="white">
+      <material name="orange">
         <color rgba="1 1 1 1"/>
       </material>
@@ -111,5 +111,5 @@
       </geometry>
       <origin xyz="0 0.111 0.102"/>
-      <material name="white">
+      <material name="orange">
         <color rgba="1 1 1 1"/>
       </material>
@@ -145,5 +145,5 @@
       </geometry>
       <origin xyz="0 0 0"/>
-      <material name="white">
+      <material name="orange">
         <color rgba="1 1 1 1"/>
       </material>
@@ -177,5 +177,5 @@
       </geometry>
       <origin xyz="-0.0275 0 0"/>
-      <material name="white">
+      <material name="orange">
         <color rgba="1 1 1 1"/>
       </material>
@@ -211,5 +211,5 @@
       </geometry>
       <origin xyz="0 0 0.1815"/>
-      <material name="white">
+      <material name="orange">
         <color rgba="1 1 1 1"/>
       </material>
@@ -245,5 +245,5 @@
       </geometry>
       <origin xyz="0 0 0"/>
-      <material name="white">
+      <material name="orange">
         <color rgba="1 1 1 1"/>
       </material>
@@ -279,5 +279,5 @@
       </geometry>
       <origin xyz="0 0 0.0325"/>
-      <material name="white">
+      <material name="orange">
         <color rgba="1 1 1 1"/>
       </material>
@@ -288,5 +288,5 @@
       </geometry>
       <origin xyz="0 0 0.0325"/>
-      <material name="white">
+      <material name="orange">
         <color rgba="1 1 1 1"/>
       </material>

Commit message: added new gripper links

File: mitsubishi_arm_description/robots/mitsubishi_rv_6sdl.urdf.xacro (robot description, xacro)
@@ -82,4 +82,66 @@
     </inertial>
   </link>
+  <joint name="finger_2_joint" type="fixed">
+    <parent link="finger_1"/>
+    <child link="finger_2"/>
+    <origin xyz="0.17 0 0.12"  rpy="0 1.56 0"/> <!-- original is 0.085 but we have the torque sensor...-->
+    <dynamics damping="100.0" friction="100.0" />
+  </joint>
+  <link name="finger_2">
+    <visual>
+     <geometry>
+	<box size="0.2 .05 .02"/>
+      </geometry>
+      <origin xyz="0 0 -0.011"/>
+      <material name="orange">
+        <color rgba="1 1 1 1"/>
+      </material>
+    </visual>
+    <collision>
+     <geometry>
+	<box size="0.1 .05 .02"/>
+      </geometry>
+      <origin xyz="0 0 -0.011"/>
+    </collision>
+    <inertial>
+      <origin xyz="0 0 1" rpy="0 0 0"/>
+      <mass value="0.01"/>
+      <inertia
+        ixx="1.0" ixy="0.0" ixz="0.0"
+        iyy="1.0" iyz="0.0"
+        izz="1.0"/>
+    </inertial>
+  </link>
+  <joint name="finger_3_joint" type="fixed">
+    <parent link="finger_1"/>
+    <child link="finger_3"/>
+    <origin xyz="-0.17 0 0.12"  rpy="0 1.56 0"/> <!-- original is 0.085 but we have the torque sensor...-->
+    <dynamics damping="100.0" friction="100.0" />
+  </joint>
+  <link name="finger_3">
+    <visual>
+     <geometry>
+	<box size="0.2 .05 .02"/>
+      </geometry>
+      <origin xyz="0 0 -0.011"/>
+      <material name="orange">
+        <color rgba="1 1 1 1"/>
+      </material>
+    </visual>
+    <collision>
+     <geometry>
+	<box size="0.1 .05 .02"/>
+      </geometry>
+      <origin xyz="0 0 -0.011"/>
+    </collision>
+    <inertial>
+      <origin xyz="0 0 1" rpy="0 0 0"/>
+      <mass value="0.01"/>
+      <inertia
+        ixx="1.0" ixy="0.0" ixz="0.0"
+        iyy="1.0" iyz="0.0"
+        izz="1.0"/>
+    </inertial>
+  </link>
   <!-- Kinect -->
   <!--<xacro:include filename="$(find mitsubishi_arm_description)/urdf/sensors.xacro" />-->

Commit message: minor changes in the calibration package

File: mitsubishi_arm_description/robots/mitsubishi_rv_6sdl.urdf.xacro (robot description, xacro)
@@ -162,5 +162,5 @@
   <!-- Transformation from the arm base to the kinect base link -->
   <xacro:kinect_camera_v0 name="camera" parent="base_link" >
-     <origin xyz="0.796357 0.919602 0.431341" rpy="0.0247013 0.415733 -1.55723"/>
+     <origin xyz="0.810223 0.920646 0.424889" rpy="0.0137265 0.405234 -1.5458"/>
   </xacro:kinect_camera_v0 >
 </robot>
