Commit message: - Modified the calibration to calibrate in -y direction and the description file to add the barrett hand

File: mitsubishi_arm_description/robots/mitsubishi_rv_6sdl.urdf.xacro (robot description, xacro)
@@ -30,5 +30,11 @@
   <!-- LINKS   -->
   <xacro:include filename="$(find mitsubishi_arm_description)/urdf/mitsubishi_rv_6sdl_arm.xacro" />
+  <xacro:include filename="$(find bhand_description)/urdf/bh282.urdf.xacro" />
+  <xacro:bhand_macro name="bh" parent="end_effector">
+	<origin xyz="0 0 0" rpy="0 0 0" />
+  </xacro:bhand_macro>
 `
+  <!-- *********************commented to add the barrett hand**********************-->
+  <!--
   <joint name="end_effector_to_gripper_palm" type="fixed">
     <axis xyz="0 0 1"/>
@@ -36,9 +42,10 @@
     <parent link="end_effector"/>
     <child link="palm_frame"/>
-    <origin xyz="0 0 0.065"  rpy="0 0 0"/> <!-- original is 0.085 but we have the torque sensor...-->
-   <dynamics damping="100.0" friction="100.0" />
+    <origin xyz="0 0 0.065"  rpy="0 0 0"/> --><!-- original is 0.085 but we have the torque sensor...-->
+<!--   <dynamics damping="100.0" friction="100.0" />
   </joint>
+  -->
   <!-- end_effector -->
-  <link name="palm_frame">
+ <!-- <link name="palm_frame">
     <inertial>
       <origin xyz="0 0 1" rpy="0 0 0"/>
@@ -54,6 +61,6 @@
     <parent link="palm_frame"/>
     <child link="finger_1"/>
-    <origin xyz="0 0 0"  rpy="0 0 1.56"/> <!-- original is 0.085 but we have the torque sensor...-->
-   <dynamics damping="100.0" friction="100.0" />
+    <origin xyz="0 0 0"  rpy="0 0 1.56"/> --><!-- original is 0.085 but we have the torque sensor...-->
+<!--   <dynamics damping="100.0" friction="100.0" />
   </joint>
   <link name="finger_1">
@@ -85,6 +92,6 @@
     <parent link="finger_1"/>
     <child link="finger_2"/>
-    <origin xyz="0.17 0 0.12"  rpy="0 1.56 0"/> <!-- original is 0.085 but we have the torque sensor...-->
-    <dynamics damping="100.0" friction="100.0" />
+    <origin xyz="0.17 0 0.12"  rpy="0 1.56 0"/> --><!-- original is 0.085 but we have the torque sensor...-->
+<!--    <dynamics damping="100.0" friction="100.0" />
   </joint>
   <link name="finger_2">
@@ -116,6 +123,6 @@
     <parent link="finger_1"/>
     <child link="finger_3"/>
-    <origin xyz="-0.17 0 0.12"  rpy="0 1.56 0"/> <!-- original is 0.085 but we have the torque sensor...-->
-    <dynamics damping="100.0" friction="100.0" />
+    <origin xyz="-0.17 0 0.12"  rpy="0 1.56 0"/> --><!-- original is 0.085 but we have the torque sensor...-->
+  <!--  <dynamics damping="100.0" friction="100.0" />
   </joint>
   <link name="finger_3">
@@ -144,4 +151,14 @@
     </inertial>
   </link>
+ -->
+   <!-- *******************************************-->
+  <!-- Kinect -->
+  <!--<xacro:include filename="$(find mitsubishi_arm_description)/urdf/sensors.xacro" />-->
+  <!-- kinect to base link -->
+ <!-- <joint name="camera_in_world_joint" type="fixed">
+    <parent link="base_link"/>
+    <child link="camera_link"/>
+    <origin xyz="0.796357 0.919602 0.431341" rpy="0.0247013 0.415733 -1.55723"/>
+  </joint>  -->
   <!-- Kinect -->
   <!--<xacro:include filename="$(find mitsubishi_arm_description)/urdf/sensors.xacro" />-->
@@ -162,5 +179,5 @@
   <!-- Transformation from the arm base to the kinect base link -->
   <xacro:kinect_camera_v0 name="camera" parent="base_link" >
-     <origin xyz="0.810223 0.920646 0.424889" rpy="0.0137265 0.405234 -1.5458"/>
+     <origin xyz="0.537566 -0.979771 0.436556" rpy="0.00848366 0.240007 1.585"/>
   </xacro:kinect_camera_v0 >
 </robot>

File: mitsubishi_arm_description/urdf/sensors.urdf.xacro (robot description, xacro)
@@ -20,5 +20,5 @@
       </inertial>
       <visual>
-        <origin xyz="0.0 0.012 0" rpy="0 0 0"/>
+	<origin xyz="0.0 0.012 0" rpy="0 0 0"/>
         <geometry>
           <mesh filename="package://pr2_description/meshes/sensors/kinect_v0/kinect.dae" scale="0.001 0.001 0.001" />
@@ -33,5 +33,5 @@
     </link>
     <joint name="${name}_optical_joint" type="fixed">
-      <origin xyz="${cal_kinect_x}            ${cal_kinect_y}         ${cal_kinect_z}"
+      <origin xyz="${cal_kinect_x}           ${cal_kinect_y}         ${cal_kinect_z}"
                 rpy="${-M_PI/2+cal_kinect_roll} ${0.0+cal_kinect_pitch} ${-M_PI/2+cal_kinect_yaw}" />
       <parent link="${name}_link"/>

Commit message: - restoring gazebo simulation functionalities

File: mitsubishi_arm_description/robots/mitsubishi_rv_6sdl.urdf.xacro (robot description, xacro)
@@ -154,11 +154,11 @@
    <!-- *******************************************-->
   <!-- Kinect -->
-  <!--<xacro:include filename="$(find mitsubishi_arm_description)/urdf/sensors.xacro" />-->
+  <xacro:include filename="$(find mitsubishi_arm_description)/urdf/sensors.xacro" />
   <!-- kinect to base link -->
- <!-- <joint name="camera_in_world_joint" type="fixed">
+ <joint name="camera_in_world_joint" type="fixed">
     <parent link="base_link"/>
     <child link="camera_link"/>
     <origin xyz="0.796357 0.919602 0.431341" rpy="0.0247013 0.415733 -1.55723"/>
-  </joint>  -->
+  </joint>
   <!-- Kinect -->
   <!--<xacro:include filename="$(find mitsubishi_arm_description)/urdf/sensors.xacro" />-->

File: mitsubishi_arm_description/urdf/mitsubishi_rv_6sdl_arm.xacro (robot description, xacro)
@@ -322,5 +322,7 @@
   <transmission name="tran1">
     <type>transmission_interface/SimpleTransmission</type>
-    <joint name="j1"/>
+    <joint name="j1">
+      <hardwareInterface>PositionJointInterface</hardwareInterface>
+    </joint>
     <actuator name="motor1">
       <hardwareInterface>EffortJointInterface</hardwareInterface>
@@ -330,5 +332,7 @@
   <transmission name="tran2">
     <type>transmission_interface/SimpleTransmission</type>
-    <joint name="j2"/>
+    <joint name="j2">
+      <hardwareInterface>PositionJointInterface</hardwareInterface>
+    </joint>
     <actuator name="motor2">
       <hardwareInterface>EffortJointInterface</hardwareInterface>
@@ -338,5 +342,7 @@
   <transmission name="tran3">
     <type>transmission_interface/SimpleTransmission</type>
-    <joint name="j3"/>
+    <joint name="j3">
+      <hardwareInterface>PositionJointInterface</hardwareInterface>
+    </joint>
     <actuator name="motor3">
       <hardwareInterface>EffortJointInterface</hardwareInterface>
@@ -346,5 +352,7 @@
   <transmission name="tran4">
     <type>transmission_interface/SimpleTransmission</type>
-    <joint name="j4"/>
+    <joint name="j4">
+      <hardwareInterface>PositionJointInterface</hardwareInterface>
+    </joint>
     <actuator name="motor4">
       <hardwareInterface>EffortJointInterface</hardwareInterface>
@@ -354,5 +362,7 @@
   <transmission name="tran5">
     <type>transmission_interface/SimpleTransmission</type>
-    <joint name="j5"/>
+    <joint name="j5">
+      <hardwareInterface>PositionJointInterface</hardwareInterface>
+    </joint>
     <actuator name="motor5">
       <hardwareInterface>EffortJointInterface</hardwareInterface>
@@ -362,5 +372,7 @@
   <transmission name="tran6">
     <type>transmission_interface/SimpleTransmission</type>
-    <joint name="j6"/>
+    <joint name="j6">
+      <hardwareInterface>PositionJointInterface</hardwareInterface>
+    </joint>
     <actuator name="motor6">
       <hardwareInterface>EffortJointInterface</hardwareInterface>

File: mitsubishi_arm_description/urdf/sensors.gazebo.xacro (robot description, xacro)
@@ -30,9 +30,9 @@
         <frameName>${name}_optical_frame</frameName>
         <pointCloudCutoff>0.5</pointCloudCutoff>
-        <distortionK1>0.00000001</distortionK1>
-        <distortionK2>0.00000001</distortionK2>
-        <distortionK3>0.00000001</distortionK3>
-        <distortionT1>0.00000001</distortionT1>
-        <distortionT2>0.00000001</distortionT2>
+        <distortionK1>0.0000000</distortionK1>
+        <distortionK2>0.0000000</distortionK2>
+        <distortionK3>0.0000000</distortionK3>
+        <distortionT1>0.0000000</distortionT1>
+        <distortionT2>0.0000000</distortionT2>
         <CxPrime>0</CxPrime>
         <Cx>0</Cx>
@@ -68,9 +68,9 @@
         <frameName>${name}_optical_frame</frameName>
         <pointCloudCutoff>0.5</pointCloudCutoff>
-        <distortionK1>0.00000001</distortionK1>
-        <distortionK2>0.00000001</distortionK2>
-        <distortionK3>0.00000001</distortionK3>
-        <distortionT1>0.00000001</distortionT1>
-        <distortionT2>0.00000001</distortionT2>
+        <distortionK1>0.0000000</distortionK1>
+        <distortionK2>0.0000000</distortionK2>
+        <distortionK3>0.0000000</distortionK3>
+        <distortionT1>0.0000000</distortionT1>
+        <distortionT2>0.0000000</distortionT2>
         <CxPrime>0</CxPrime>
         <Cx>0</Cx>

Commit message: - changed the limit of the last joint j6 from 360 to 180 and commented some parts

File: mitsubishi_arm_description/robots/mitsubishi_rv_6sdl.urdf.xacro (robot description, xacro)
@@ -30,10 +30,17 @@
   <!-- LINKS   -->
   <xacro:include filename="$(find mitsubishi_arm_description)/urdf/mitsubishi_rv_6sdl_arm.xacro" />
-  <xacro:include filename="$(find bhand_description)/urdf/bh282.urdf.xacro" />
-  <xacro:bhand_macro name="bh" parent="end_effector">
+  <!-- **********************barret hand part (old)****************************** -->
+  <!-- xacro:include filename="$(find bhand_description)/urdf/bh280.urdf.xacro" / -->
+  <!-- xacro:bhand_macro name="bh" parent="end_effector">
 	<origin xyz="0 0 0" rpy="0 0 0" />
-  </xacro:bhand_macro>
-`
-  <!-- *********************commented to add the barrett hand**********************-->
+  </xacro:bhand_macro -->
+` <!-- *************************************************************************** -->
+  <!-- **********************barret hand part (new)****************************** -->
+<!--  <xacro:include filename="$(find barrett_hand_description)/urdf/barrett_hand.xacro" />
+  <joint name="barrett_hand_base_link" type="fixed">
+  <parent link="end_effector"/>
+  <child link="barrett_base_link"/>
+  </joint>-->
+` <!-- ************************************************************************** -->
   <!--
   <joint name="end_effector_to_gripper_palm" type="fixed">
@@ -153,12 +160,13 @@
  -->
    <!-- *******************************************-->
-  <!-- Kinect -->
-  <xacro:include filename="$(find mitsubishi_arm_description)/urdf/sensors.xacro" />
+   <!-- Kinect -->
+<!--  <xacro:include filename="$(find mitsubishi_arm_description)/urdf/sensors.xacro" />-->
   <!-- kinect to base link -->
- <joint name="camera_in_world_joint" type="fixed">
+ <!--<joint name="camera_in_world_joint" type="fixed">
     <parent link="base_link"/>
     <child link="camera_link"/>
     <origin xyz="0.796357 0.919602 0.431341" rpy="0.0247013 0.415733 -1.55723"/>
   </joint>
+  -->
   <!-- Kinect -->
   <!--<xacro:include filename="$(find mitsubishi_arm_description)/urdf/sensors.xacro" />-->
@@ -179,5 +187,6 @@
   <!-- Transformation from the arm base to the kinect base link -->
   <xacro:kinect_camera_v0 name="camera" parent="base_link" >
-     <origin xyz="0.537566 -0.979771 0.436556" rpy="0.00848366 0.240007 1.585"/>
+    <!-- origin xyz="0.537566 -0.979771 0.436556" rpy="0.00848366 0.240007 1.585"/ --> <!-- camera is to the mitsubishi left -->
+    <origin xyz="0.691031 0.995553 0.428516" rpy="0.00123993 0.231118 -1.56538"/> <!-- camera is to the mitsubishi right (previous location) -->
   </xacro:kinect_camera_v0 >
 </robot>

File: mitsubishi_arm_description/urdf/mitsubishi_rv_6sdl_arm.xacro (robot description, xacro)
@@ -266,5 +266,5 @@
   <joint name="j6" type="revolute">
     <axis xyz="0 0 1"/>
-    <limit effort="1000.0" lower="${(-360+offset_from_limit)*PI/180}" upper="${(360-offset_from_limit)*PI/180}" velocity="0.2"/>
+    <limit effort="1000.0" lower="${(-180+offset_from_limit)*PI/180}" upper="${(180-offset_from_limit)*PI/180}" velocity="0.2"/><!-- instead of -180 is -360 , 180 is 360 -->
     <parent link="wrist"/>
     <child link="torque_sensor"/>
