Commit message: mitsubishi config files changed

File: mitsubishi_arm_description/urdf/mitsubishi_rv_6sdl_arm.urdf.xacro (robot description, xacro)
@@ -20,5 +20,5 @@
   <joint name="j1" type="revolute">
     <axis xyz="0 0 1"/>
-    <limit effort="1000.0" lower="-3.10668606855" upper="3.10668606855" velocity="0.5"/>
+    <limit effort="1000.0" lower="-2.96" upper="2.96" velocity="0.5"/>
     <parent link="base_link"/>
     <child link="shoulder_block"/>
@@ -44,5 +44,5 @@
   <joint name="j2" type="revolute">
     <axis xyz="0 0 1"/>
-    <limit effort="1000.0" lower="-2.75762021815" upper="2.75762021815" velocity="0.5"/>
+    <limit effort="1000.0" lower="-1.6" upper="2.35" velocity="0.5"/>
     <parent link="shoulder_block"/>
     <child link="shoulder"/>

Commit message: re-added mitsubishi packages after accidentally removing them

File: mitsubishi_arm_description/urdf/mitsubishi_rv_6sdl_arm.urdf.xacro (robot description, xacro)
@@ -20,5 +20,5 @@
   <joint name="j1" type="revolute">
     <axis xyz="0 0 1"/>
-    <limit effort="1000.0" lower="-2.96" upper="2.96" velocity="0.5"/>
+    <limit effort="1000.0" lower="-3.10668606855" upper="3.10668606855" velocity="0.5"/>
     <parent link="base_link"/>
     <child link="shoulder_block"/>
@@ -44,8 +44,8 @@
   <joint name="j2" type="revolute">
     <axis xyz="0 0 1"/>
-    <limit effort="1000.0" lower="-1.6" upper="2.35" velocity="0.5"/>
+    <limit effort="1000.0" lower="-2.75762021815" upper="2.75762021815" velocity="0.5"/>
     <parent link="shoulder_block"/>
     <child link="shoulder"/>
-    <origin xyz="0.085 0 0.111" rpy="1.57079632679 0 0"/>
+    <origin xyz="0.085 0 0.111" rpy="1.57079632679 0 3.14159265359"/>
   </joint>
   <link name="shoulder">
@@ -95,5 +95,5 @@
     <parent link="upper_arm"/>
     <child link="elbow"/>
-    <origin xyz="0 0.295 0"/>
+    <origin xyz="0 0.295 0" rpy="3.14159265359 0 1.57"/>
   </joint>
   <link name="elbow">
@@ -165,5 +165,5 @@
     <parent link="fore_arm"/>
     <child link="wrist"/>
-    <origin xyz="0 0 0.240"  rpy="0 -1.5707963267 0"/>
+    <origin xyz="0 0 0.240"  rpy="3.14159265359 -1.5707963267 0"/>
   </joint>
   <link name="wrist">

Commit message: added new  barret hand packages including description, msgs and control (still need to clean the package). Added also some mitsubishi related missing files

File: mitsubishi_arm_description/urdf/mitsubishi_rv_6sdl_arm.urdf.xacro (robot description, xacro)
@@ -1,4 +1,5 @@
 <?xml version="1.0"?>
 <robot xmlns:xacro="http://www.ros.org/wiki/xacro">
+  <property name="PI" value="3.1415926535897931" />
   <link name="base_link" >
     <visual>
@@ -20,5 +21,5 @@
   <joint name="j1" type="revolute">
     <axis xyz="0 0 1"/>
-    <limit effort="1000.0" lower="-3.10668606855" upper="3.10668606855" velocity="0.5"/>
+    <limit effort="1000.0" lower="${-169*PI/180}" upper="${169*PI/180}" velocity="0.5"/>
     <parent link="base_link"/>
     <child link="shoulder_block"/>
@@ -44,5 +45,5 @@
   <joint name="j2" type="revolute">
     <axis xyz="0 0 1"/>
-    <limit effort="1000.0" lower="-2.75762021815" upper="2.75762021815" velocity="0.5"/>
+    <limit effort="1000.0" lower="${-92*PI/180}" upper="${131*PI/180}" velocity="0.5"/>
     <parent link="shoulder_block"/>
     <child link="shoulder"/>
@@ -68,5 +69,4 @@
   <joint name="fixed_joint_1" type="fixed">
     <axis xyz="0 0 1"/>
-    <limit effort="1000.0" lower="0.0" upper="2.18166156499" velocity="0.5"/>
     <parent link="shoulder"/>
     <child link="upper_arm"/>
@@ -92,5 +92,5 @@
   <joint name="j3" type="revolute">
     <axis xyz="0 0 1"/>
-    <limit effort="1000.0" lower="-2.75762021815" upper="2.75762021815" velocity="0.5"/>
+    <limit effort="1000.0" lower="${-128*PI/180}" upper="${165*PI/180}" velocity="0.5"/>
     <parent link="upper_arm"/>
     <child link="elbow"/>
@@ -138,5 +138,5 @@
   <joint name="j4" type="revolute">
     <axis xyz="0 0 1"/>
-    <limit effort="1000.0" lower="0.0" upper="2.18166156499" velocity="0.5"/>
+    <limit effort="1000.0" lower="${-159*PI/180}" upper="${159*PI/180}" velocity="0.5"/>
     <parent link="elbow_block"/>
     <child link="fore_arm"/>
@@ -162,5 +162,5 @@
   <joint name="j5" type="revolute">
     <axis xyz="0 0 1"/>
-    <limit effort="1000.0" lower="-0.92502450355" upper="0.92502450355" velocity="0.5"/>
+    <limit effort="1000.0" lower="${-110*PI/180}" upper="${110*PI/180}" velocity="0.5"/>
     <parent link="fore_arm"/>
     <child link="wrist"/>
@@ -186,5 +186,5 @@
   <joint name="j6" type="revolute">
     <axis xyz="0 0 1"/>
-    <limit effort="1000.0" lower="0.0" upper="2.18166156499" velocity="0.5"/>
+    <limit effort="1000.0" lower="${-359*PI/180}" upper="${359*PI/180}" velocity="0.5"/>
     <parent link="wrist"/>
     <child link="end_effector"/>

Commit message: mitsubishi arm is now completely integrated with MoveIt!

File: mitsubishi_arm_description/urdf/mitsubishi_rv_6sdl_arm.urdf.xacro (robot description, xacro)
@@ -2,4 +2,5 @@
 <robot xmlns:xacro="http://www.ros.org/wiki/xacro">
   <property name="PI" value="3.1415926535897931" />
+  <property name="offset_from_limit" value="5.0" />
   <link name="base_link" >
     <visual>
@@ -21,5 +22,5 @@
   <joint name="j1" type="revolute">
     <axis xyz="0 0 1"/>
-    <limit effort="1000.0" lower="${-169*PI/180}" upper="${169*PI/180}" velocity="0.5"/>
+    <limit effort="1000.0" lower="${(-170+offset_from_limit)*PI/180}" upper="${(170-offset_from_limit)*PI/180}" velocity="0.5"/>
     <parent link="base_link"/>
     <child link="shoulder_block"/>
@@ -45,5 +46,5 @@
   <joint name="j2" type="revolute">
     <axis xyz="0 0 1"/>
-    <limit effort="1000.0" lower="${-92*PI/180}" upper="${131*PI/180}" velocity="0.5"/>
+    <limit effort="1000.0" lower="${-92*PI/180}" upper="${(135-offset_from_limit)*PI/180}" velocity="0.5"/>
     <parent link="shoulder_block"/>
     <child link="shoulder"/>
@@ -78,5 +79,5 @@
 	<box size="0.090 0.210 0.02"/>
       </geometry>
-      <origin xyz="0 0.105 -0.102"/>
+      <origin xyz="0 0.105 0.102"/>
       <material name="white">
         <color rgba="1 1 1 1"/>
@@ -92,8 +93,8 @@
   <joint name="j3" type="revolute">
     <axis xyz="0 0 1"/>
-    <limit effort="1000.0" lower="${-128*PI/180}" upper="${165*PI/180}" velocity="0.5"/>
+    <limit effort="1000.0" lower="${(-129+offset_from_limit)*PI/180}" upper="${(166-offset_from_limit)*PI/180}" velocity="0.5"/>
     <parent link="upper_arm"/>
     <child link="elbow"/>
-    <origin xyz="0 0.295 0" rpy="3.14159265359 0 1.57"/>
+    <origin xyz="0 0.295 0" rpy="0 0 1.57"/>
   </joint>
   <link name="elbow">
@@ -117,5 +118,5 @@
     <parent link="elbow"/>
     <child link="elbow_block"/>
-    <origin xyz="0 0.100 0"/>
+    <origin xyz="0 -0.100 0"/>
   </joint>
   <link name="elbow_block">
@@ -138,5 +139,5 @@
   <joint name="j4" type="revolute">
     <axis xyz="0 0 1"/>
-    <limit effort="1000.0" lower="${-159*PI/180}" upper="${159*PI/180}" velocity="0.5"/>
+    <limit effort="1000.0" lower="${(-160+offset_from_limit)*PI/180}" upper="${(160-offset_from_limit)*PI/180}" velocity="0.5"/>
     <parent link="elbow_block"/>
     <child link="fore_arm"/>
@@ -162,8 +163,8 @@
   <joint name="j5" type="revolute">
     <axis xyz="0 0 1"/>
-    <limit effort="1000.0" lower="${-110*PI/180}" upper="${110*PI/180}" velocity="0.5"/>
+    <limit effort="1000.0" lower="${(-110+offset_from_limit)*PI/180}" upper="${(110-offset_from_limit)*PI/180}" velocity="0.5"/>
     <parent link="fore_arm"/>
     <child link="wrist"/>
-    <origin xyz="0 0 0.240"  rpy="3.14159265359 -1.5707963267 0"/>
+    <origin xyz="0 0 0.240"  rpy="0.0 -1.5707963267 0"/>
   </joint>
   <link name="wrist">
@@ -186,5 +187,5 @@
   <joint name="j6" type="revolute">
     <axis xyz="0 0 1"/>
-    <limit effort="1000.0" lower="${-359*PI/180}" upper="${359*PI/180}" velocity="0.5"/>
+    <limit effort="1000.0" lower="${(-360+offset_from_limit)*PI/180}" upper="${(360-offset_from_limit)*PI/180}" velocity="0.5"/>
     <parent link="wrist"/>
     <child link="end_effector"/>

Commit message: MoveIt! reconfigured to work properly with mitsubishi arm

File: mitsubishi_arm_description/urdf/mitsubishi_rv_6sdl_arm.urdf.xacro (robot description, xacro)
@@ -22,5 +22,5 @@
   <joint name="j1" type="revolute">
     <axis xyz="0 0 1"/>
-    <limit effort="1000.0" lower="${(-170+offset_from_limit)*PI/180}" upper="${(170-offset_from_limit)*PI/180}" velocity="0.5"/>
+    <limit effort="1000.0" lower="${(-170+offset_from_limit)*PI/180}" upper="${(170-offset_from_limit)*PI/180}" velocity="0.05"/>
     <parent link="base_link"/>
     <child link="shoulder_block"/>
@@ -46,5 +46,5 @@
   <joint name="j2" type="revolute">
     <axis xyz="0 0 1"/>
-    <limit effort="1000.0" lower="${-92*PI/180}" upper="${(135-offset_from_limit)*PI/180}" velocity="0.5"/>
+    <limit effort="1000.0" lower="${-92*PI/180}" upper="${(135-offset_from_limit)*PI/180}" velocity="0.05"/>
     <parent link="shoulder_block"/>
     <child link="shoulder"/>
@@ -93,5 +93,5 @@
   <joint name="j3" type="revolute">
     <axis xyz="0 0 1"/>
-    <limit effort="1000.0" lower="${(-129+offset_from_limit)*PI/180}" upper="${(166-offset_from_limit)*PI/180}" velocity="0.5"/>
+    <limit effort="1000.0" lower="${(-129+offset_from_limit)*PI/180}" upper="${(166-offset_from_limit)*PI/180}" velocity="0.05"/>
     <parent link="upper_arm"/>
     <child link="elbow"/>
@@ -139,5 +139,5 @@
   <joint name="j4" type="revolute">
     <axis xyz="0 0 1"/>
-    <limit effort="1000.0" lower="${(-160+offset_from_limit)*PI/180}" upper="${(160-offset_from_limit)*PI/180}" velocity="0.5"/>
+    <limit effort="1000.0" lower="${(-160+offset_from_limit)*PI/180}" upper="${(160-offset_from_limit)*PI/180}" velocity="0.05"/>
     <parent link="elbow_block"/>
     <child link="fore_arm"/>
@@ -163,5 +163,5 @@
   <joint name="j5" type="revolute">
     <axis xyz="0 0 1"/>
-    <limit effort="1000.0" lower="${(-110+offset_from_limit)*PI/180}" upper="${(110-offset_from_limit)*PI/180}" velocity="0.5"/>
+    <limit effort="1000.0" lower="${(-110+offset_from_limit)*PI/180}" upper="${(110-offset_from_limit)*PI/180}" velocity="0.05"/>
     <parent link="fore_arm"/>
     <child link="wrist"/>
@@ -187,5 +187,5 @@
   <joint name="j6" type="revolute">
     <axis xyz="0 0 1"/>
-    <limit effort="1000.0" lower="${(-360+offset_from_limit)*PI/180}" upper="${(360-offset_from_limit)*PI/180}" velocity="0.5"/>
+    <limit effort="1000.0" lower="${(-360+offset_from_limit)*PI/180}" upper="${(360-offset_from_limit)*PI/180}" velocity="0.05"/>
     <parent link="wrist"/>
     <child link="end_effector"/>

Commit message: mitsubishi arm model now includes the torque sensor

File: mitsubishi_arm_description/urdf/mitsubishi_rv_6sdl_arm.urdf.xacro (robot description, xacro)
@@ -49,19 +49,19 @@
     <parent link="shoulder_block"/>
     <child link="shoulder"/>
-    <origin xyz="0.085 0 0.111" rpy="1.57079632679 0 3.14159265359"/>
+    <origin xyz="0.079 0 0.111" rpy="1.57079632679 0 3.14159265359"/>
   </joint>
   <link name="shoulder">
     <visual>
       <geometry>
-	<cylinder length="0.327" radius="0.085"/>
-      </geometry>
-      <origin xyz="0 0 0"/>
-      <material name="white">
-        <color rgba="1 1 1 1"/>
-      </material>
-    </visual>
-    <collision>
-      <geometry>
-        <cylinder length="0.327" radius="0.085"/>
+	<cylinder length="0.327" radius="0.079"/>
+      </geometry>
+      <origin xyz="0 0 0"/>
+      <material name="white">
+        <color rgba="1 1 1 1"/>
+      </material>
+    </visual>
+    <collision>
+      <geometry>
+        <cylinder length="0.327" radius="0.079"/>
       </geometry>
       <origin xyz="0 0 0"/>
@@ -72,21 +72,21 @@
     <parent link="shoulder"/>
     <child link="upper_arm"/>
-    <origin xyz="0 0.085 0"/>
+    <origin xyz="0 0.079 0"/>
   </joint>
   <link name="upper_arm">
     <visual>
       <geometry>
-	<box size="0.090 0.210 0.02"/>
-      </geometry>
-      <origin xyz="0 0.105 0.102"/>
-      <material name="white">
-        <color rgba="1 1 1 1"/>
-      </material>
-    </visual>
-    <collision>
-      <geometry>
-	<box size="0.090 0.110 0.02"/>
-      </geometry>
-      <origin xyz="0 0.19 -0.102"/>
+	<box size="0.090 0.222 0.02"/>
+      </geometry>
+      <origin xyz="0 0.111 0.102"/>
+      <material name="white">
+        <color rgba="1 1 1 1"/>
+      </material>
+    </visual>
+    <collision>
+      <geometry>
+	<box size="0.090 0.222 0.02"/>
+      </geometry>
+      <origin xyz="0 0.111 0.102"/>
     </collision>
   </link>
@@ -96,19 +96,19 @@
     <parent link="upper_arm"/>
     <child link="elbow"/>
-    <origin xyz="0 0.295 0" rpy="0 0 1.57"/>
+    <origin xyz="0 0.301 0" rpy="0 0 1.57"/>
   </joint>
   <link name="elbow">
     <visual>
       <geometry>
-	<cylinder length="0.327" radius="0.085"/>
-      </geometry>
-      <origin xyz="0 0 0"/>
-      <material name="white">
-        <color rgba="1 1 1 1"/>
-      </material>
-    </visual>
-    <collision>
-      <geometry>
-        <cylinder length="0.327" radius="0.085"/>
+	<cylinder length="0.327" radius="0.079"/>
+      </geometry>
+      <origin xyz="0 0 0"/>
+      <material name="white">
+        <color rgba="1 1 1 1"/>
+      </material>
+    </visual>
+    <collision>
+      <geometry>
+        <cylinder length="0.327" radius="0.079"/>
       </geometry>
       <origin xyz="0 0 0"/>
@@ -142,21 +142,21 @@
     <parent link="elbow_block"/>
     <child link="fore_arm"/>
-    <origin xyz="0.085 0 0"  rpy="0 1.5707963267 0"/>
+    <origin xyz="0.079 0 0"  rpy="0 1.5707963267 0"/>
   </joint>
   <link name="fore_arm">
     <visual>
       <geometry>
-	<box size="0.170 .120 .230"/>
-      </geometry>
-      <origin xyz="0 0 0.115"/>
-      <material name="white">
-        <color rgba="1 1 1 1"/>
-      </material>
-    </visual>
-    <collision>
-      <geometry>
-	<box size="0.225 .126 .239"/>
-      </geometry>
-      <origin xyz="-0.0275 0 0"/>
+	<box size="0.170 .120 .346"/>
+      </geometry>
+      <origin xyz="0 0 0.1815"/>
+      <material name="white">
+        <color rgba="1 1 1 1"/>
+      </material>
+    </visual>
+    <collision>
+      <geometry>
+	<box size="0.170 .120 .346"/>
+      </geometry>
+      <origin xyz="0 0 0.1815"/>
     </collision>
   </link>
@@ -166,5 +166,5 @@
     <parent link="fore_arm"/>
     <child link="wrist"/>
-    <origin xyz="0 0 0.240"  rpy="0.0 -1.5707963267 0"/>
+    <origin xyz="0 0 0.346"  rpy="0.0 -1.5707963267 0"/>
   </joint>
   <link name="wrist">
@@ -189,6 +189,30 @@
     <limit effort="1000.0" lower="${(-360+offset_from_limit)*PI/180}" upper="${(360-offset_from_limit)*PI/180}" velocity="0.05"/>
     <parent link="wrist"/>
+    <child link="torque_sensor"/>
+    <origin xyz="0.085 0 0"  rpy="0 1.5707963267 0"/>
+  </joint>
+  <link name="torque_sensor">
+    <visual>
+     <geometry>
+	<cylinder  length="0.065" radius="0.035"/>
+      </geometry>
+      <origin xyz="0 0 0.0325"/>
+      <material name="white">
+        <color rgba="1 1 1 1"/>
+      </material>
+    </visual>
+    <collision>
+     <geometry>
+	<box size="0.02 .02 0.065"/>
+      </geometry>
+      <origin xyz="0 0 0.065"/>
+    </collision>
+  </link>
+  <joint name="torque_sensor_joint" type="fixed">
+    <axis xyz="0 0 1"/>
+    <limit effort="1000.0" lower="${(-360+offset_from_limit)*PI/180}" upper="${(360-offset_from_limit)*PI/180}" velocity="0.05"/>
+    <parent link="torque_sensor"/>
     <child link="end_effector"/>
-    <origin xyz="0.085 0 0"  rpy="0 1.5707963267 0"/>
+    <origin xyz="0 0 0.065"  rpy="0 0 0"/> <!-- original is 0.085 but we have the torque sensor...-->
   </joint>
   <link name="end_effector">

Commit message: barrett hand moveit planner is working

File: mitsubishi_arm_description/urdf/mitsubishi_rv_6sdl_arm.urdf.xacro (robot description, xacro)
@@ -204,7 +204,10 @@
     <collision>
      <geometry>
-	<box size="0.02 .02 0.065"/>
-      </geometry>
-      <origin xyz="0 0 0.065"/>
+	<cylinder  length="0.065" radius="0.035"/>
+      </geometry>
+      <origin xyz="0 0 0.0325"/>
+      <material name="white">
+        <color rgba="1 1 1 1"/>
+      </material>
     </collision>
   </link>
