Commit message: Barrett hand working in gazebo!

File: mitsubishi_arm_description/urdf/mitsubishi_rv_6sdl_arm.xacro (robot description, xacro)
@@ -31,5 +31,5 @@
   <joint name="j1" type="revolute">
     <axis xyz="0 0 1"/>
-    <limit effort="1000.0" lower="${(-170+offset_from_limit)*PI/180}" upper="${(170-offset_from_limit)*PI/180}" velocity="0.05"/>
+    <limit effort="1000.0" lower="${(-170+offset_from_limit)*PI/180}" upper="${(170-offset_from_limit)*PI/180}" velocity="0.2"/>
     <parent link="base_link"/>
     <child link="shoulder_block"/>
@@ -65,5 +65,5 @@
   <joint name="j2" type="revolute">
     <axis xyz="0 0 1"/>
-    <limit effort="1000.0" lower="${-92*PI/180}" upper="${(135-offset_from_limit)*PI/180}" velocity="0.05"/>
+    <limit effort="1000.0" lower="${-92*PI/180}" upper="${(135-offset_from_limit)*PI/180}" velocity="0.2"/>
     <parent link="shoulder_block"/>
     <child link="shoulder"/>
@@ -132,5 +132,5 @@
   <joint name="j3" type="revolute">
     <axis xyz="0 0 1"/>
-    <limit effort="1000.0" lower="${(-129+offset_from_limit)*PI/180}" upper="${(166-offset_from_limit)*PI/180}" velocity="0.05"/>
+    <limit effort="1000.0" lower="${(-129+offset_from_limit)*PI/180}" upper="${(166-offset_from_limit)*PI/180}" velocity="0.2"/>
     <parent link="upper_arm"/>
     <child link="elbow"/>
@@ -198,5 +198,5 @@
   <joint name="j4" type="revolute">
     <axis xyz="0 0 1"/>
-    <limit effort="1000.0" lower="${(-160+offset_from_limit)*PI/180}" upper="${(160-offset_from_limit)*PI/180}" velocity="0.05"/>
+    <limit effort="1000.0" lower="${(-160+offset_from_limit)*PI/180}" upper="${(160-offset_from_limit)*PI/180}" velocity="0.2"/>
     <parent link="elbow_block"/>
     <child link="fore_arm"/>
@@ -232,5 +232,5 @@
   <joint name="j5" type="revolute">
     <axis xyz="0 0 1"/>
-    <limit effort="1000.0" lower="${(-110+offset_from_limit)*PI/180}" upper="${(110-offset_from_limit)*PI/180}" velocity="0.05"/>
+    <limit effort="1000.0" lower="${(-110+offset_from_limit)*PI/180}" upper="${(110-offset_from_limit)*PI/180}" velocity="0.2"/>
     <parent link="fore_arm"/>
     <child link="wrist"/>
@@ -266,5 +266,5 @@
   <joint name="j6" type="revolute">
     <axis xyz="0 0 1"/>
-    <limit effort="1000.0" lower="${(-360+offset_from_limit)*PI/180}" upper="${(360-offset_from_limit)*PI/180}" velocity="0.05"/>
+    <limit effort="1000.0" lower="${(-360+offset_from_limit)*PI/180}" upper="${(360-offset_from_limit)*PI/180}" velocity="0.2"/>
     <parent link="wrist"/>
     <child link="torque_sensor"/>
@@ -303,5 +303,5 @@
   <joint name="torque_sensor_joint" type="fixed">
     <axis xyz="0 0 1"/>
-    <limit effort="1000.0" lower="${(-360+offset_from_limit)*PI/180}" upper="${(360-offset_from_limit)*PI/180}" velocity="0.05"/>
+    <limit effort="1000.0" lower="${(-360+offset_from_limit)*PI/180}" upper="${(360-offset_from_limit)*PI/180}" velocity="0.2"/>
     <parent link="torque_sensor"/>
     <child link="end_effector"/>
